Commit message: Got the xml working

File: tracer.urdf (robot description, URDF)
Before this commit: robot Tracer, 9 links, 8 joints
Links:
- link base_link: mass None -> 10; geometry collision box size=0.702 0.61 0.139; visual box size=0.702 0.61 0.139
- link battery: mass None -> 5; geometry collision box size=0.204978 0.37592 0.279908; visual box size=0.204978 0.37592 0.279908
- link bl_caster_wheel: mass None -> 0.2; geometry collision cylinder length=0.03 radius=0.025; visual cylinder length=0.03 radius=0.025
- link br_caster_wheel: mass None -> 0.2; geometry collision cylinder length=0.03 radius=0.025; visual cylinder length=0.03 radius=0.025
- link fl_caster_wheel: mass None -> 0.2; geometry collision cylinder length=0.03 radius=0.025; visual cylinder length=0.03 radius=0.025
- link fr_caster_wheel: mass None -> 0.2; geometry collision cylinder length=0.03 radius=0.025; visual cylinder length=0.03 radius=0.025
- link left_wheel: mass None -> 0.5; geometry collision cylinder length=0.04 radius=0.05; visual cylinder length=0.04 radius=0.05
- link lidar_link: mass None -> 0.1; geometry collision cylinder length=0.0596 radius=0.0225; visual cylinder length=0.0596 radius=0.0225
- link right_wheel: mass None -> 0.5; geometry collision cylinder length=0.04 radius=0.05; visual cylinder length=0.04 radius=0.05
